File: PCB_RAIL/PCB_RAIL.kicad_pcb (KiCad board)
At the start: 4 copper layers, 71 x 64 mm, 116 parts, among them J1 Conn_01x02, J10 Conn_01x02, J11 Conn_01x03, J12 Conn_01x03, J13 Conn_01x03, J14 Conn_01x03, J15 Conn_01x03, J16 Conn_01x03, J17 Conn_01x03, J18 Conn_01x04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

Commit message: final push readme+3d
Parts:
- removed C25: 220u, ECA1HHG471:CAPPRD500W60D1000H2000
- added C28: ECA1HHG471, ECA1HHG471:ECA1HHG471, F.Cu at (130.1, 73.0)
- C1, C9: value 220u -> ECA1HHG471; footprint ECA1HHG471:CAPPRD500W60D1000H2000 -> ECA1HHG471:ECA1HHG471
- J1: footprint Connector_AMASS:AMASS_XT30U-F_1x02_P5.0mm_Vertical -> conn_ARES:XT30-F-2P
- S2, S3: value 436331045822 -> WS-TASU SMT Tact Switch with Boss Design 4.7x3.5 mm side push
- U3: footprint Package_DFN_QFN:QFN-48-1EP_7x7mm_P0.5mm_EP5.6x5.6mm -> STM32G431CBU6:STM32G431CBU6
- moved C9 33.6 mm to (105.7, 96.2), turned to 0 degrees
- moved J1 4.87 mm to (102.5, 83.1), turned to -90 degrees
- moved C1 0.09 mm to (104.0, 73.6)
Connections:
- C9 pad 1: 24V -> +12V
- J1 pad 1: GND -> 24V
- J1 pad 2: 24V -> GND
Routing:
- net GND: track 4.42 -> 27.1 mm, vias 251 -> 249
