File: PCB_RAIL/PCB_RAIL.kicad_sch (KiCad schematic)
At the start: 51 parts, among them J1 Conn_01x02, J10 Conn_01x02, J11 Conn_01x03, J12 Conn_01x03, J13 Conn_01x03, J14 Conn_01x03, J15 Conn_01x03, J16 Conn_01x03, J17 Conn_01x03, J18 Conn_01x04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

Commit message: final push readme+3d
Parts:
- removed C1, C25, C9: 220u, ECA1HHG471:CAPPRD500W60D1000H2000, symbol Device:C_Polarized
- added C1, C28, C9: ECA1HHG471, ECA1HHG471:ECA1HHG471, symbol ECA1HHG471:ECA1HHG471
- J1: footprint Connector_AMASS:AMASS_XT30U-F_1x02_P5.0mm_Vertical -> conn_ARES:XT30-F-2P
Connections:
- net +12V: now also C9.1
- net 24V: now also J1.1 (Pin_1), C1.1, C28.1; no longer J1.2 (Pin_2)
- net GND: now also J1.2 (Pin_2), C1.2, C28.2, C9.2; no longer J1.1 (Pin_1)
Other:
- moved on the sheet: J1
