File: PCB_RAIL/µC.kicad_sch (KiCad schematic)
At the start: 27 parts, among them J20 Conn_ST_STDC14, U3 STM32G431CBUx, Y2 WE-XTAL_CFPX-104

Commit message: final push readme+3d
Parts:
- U3: footprint Package_DFN_QFN:QFN-48-1EP_7x7mm_P0.5mm_EP5.6x5.6mm -> STM32G431CBU6:STM32G431CBU6
Changed lines of the file:
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@@
 		)
 		(instances
-			(project ""
+			(project "PCB_RAIL"
 				(path "/fe9a38fd-9574-4626-83c5-735e6b11628f/3b40d16f-eabf-42fa-8d3a-54e367c9dc5b"
 					(reference "Y2")
@@
 		)
 		(instances
-			(project ""
+			(project "PCB_RAIL"
 				(path "/fe9a38fd-9574-4626-83c5-735e6b11628f/3b40d16f-eabf-42fa-8d3a-54e367c9dc5b"
 					(reference "#PWR053")
@@
 		)
 		(instances
-			(project ""
+			(project "PCB_RAIL"
 				(path "/fe9a38fd-9574-4626-83c5-735e6b11628f/3b40d16f-eabf-42fa-8d3a-54e367c9dc5b"
 					(reference "R8")
@@
 			)
 		)
-		(property "Footprint" "Package_DFN_QFN:QFN-48-1EP_7x7mm_P0.5mm_EP5.6x5.6mm"
+		(property "Footprint" "STM32G431CBU6:STM32G431CBU6"
 			(at 195.58 130.81 0)
 			(effects
